File: hw/eagle/CC3D_micro.sch (EAGLE design)
At the start: 76 parts, among them IC1 STM32F103CBT6, IC2 MPU-6050, IC3 MS5611, IC4 SPI_FLASH-X25XXSMD, IC5 MCP1703CB, U2 STM32F030XTSSOP20, Y1 8MHZ

Commit message: hw v0.2
Parts:
- removed C20: 47n, RC.v2:C0402
- added C1: u47, RC.v2:C0402
- added R1: 22, RC.v2:R0402
- C10: value 47n -> u1
- C11, C3: value 0u1 -> 47n
- C12: device RC.v2:C0603 -> RC.v2:C0402
- C13, C14: value 2u2 -> 0u1; device RC.v2:C0805 -> RC.v2:C0402
- C16: value 47n -> 0u1; device RC.v2:C0402 -> RC.v2:C0603
- C17: value 2n2 50v -> 0u1
- C18: value u47 -> 2u2; device RC.v2:C0402 -> RC.v2:C0805
- C19: value u47 -> 2u2
- C2: value 0u1 -> u47
- C5: value 0u1 -> 2n2 50v
- C6: value u1 -> 47n
- C7: value u1 -> u47; device RC.v2:C0402 -> RC.v2:C0805
- C9: value u47 -> u1
- IC1: value STM32F103CBT6 -> MPU-6050; device cc3d:STM32F103C8 -> cc3d:MPU-6050
- IC2: value MPU-6050 -> MS5611; device cc3d:MPU-6050 -> cc3d:MS5611
- IC3: value MS5611 -> MCP1703CB; device cc3d:MS5611 -> semi:MCP1703CB
- IC4: value SPI_FLASH-X25XXSMD -> STM32F103CBT6; device cc3d:SPI_FLASH-X25XXSMD -> cc3d:STM32F103C8
- IC5: value MCP1703CB -> SPI_FLASH-X25XXSMD; device semi:MCP1703CB -> cc3d:SPI_FLASH-X25XXSMD
- IC6: value STM32F030XTSSOP20 -> STM32F030F4T6
- PAD1: value (none) -> VCC
- PAD10, PAD16: value SWCLK -> (none)
- PAD11: value PPM -> (none)
- PAD12: value RX/SDA -> (none)
- PAD13: value TX/SCL -> (none)
- PAD14: value VCC -> (none)
- PAD15: value GND -> (none)
- PAD17: value SWDIO -> (none)
- PAD2: value (none) -> GND
- PAD3: value (none) -> RX/SDA
- PAD4: value (none) -> TX/SCL
- PAD5, PAD8: value (none) -> SWCLK
- PAD6: value (none) -> SWDIO
- PAD7: value (none) -> PPM
- R10: value 10k -> 1k
- R11: value 15k -> 680
- R12: value 1k -> 510
- R14: value 510 -> 10k
- R15: value 680 -> 1k
- R16: value DNP -> 680
- R2: value 10k -> 22
- R3: value 10k -> 1k5
- R5: value 2k2 -> 10k
- R6: value 680 -> 2k2
- R7: value 22 -> 10k
- R8: value 22 -> 15k
- R9: value 1k5 -> DNP
- renumbered D5 to D1, U2 to IC6
Connections:
- new net N$7: IC6.BOOT0, R10.P$1
- net BAT: now also C18.P$2, C19.P$2, PAD10.P, PAD12.P, PAD14.P, PAD16.P; no longer C13.P$2, C14.P$2, PAD3.P, PAD4.P, PAD7.P, PAD8.P
- net FLEXI_RX/SDA: now also IC2.SDI/SDA, IC4.PB11, PAD3.P, R6.P$1; no longer IC1.PB11, IC3.SDI/SDA, PAD12.P, R5.P$1
- net FLEXI_TX/SCL: now also IC2.SCLK, IC4.PB10, PAD4.P; no longer IC1.PB10, IC3.SCLK, PAD13.P
- net GND: now also C1.P$1, C10.P$2, C11.P$1, C12.P$1, C16.P$2, C17.P$2, C7.P$1, IC1.CLKIN, IC1.FSYNC, IC1.GND, IC2.CSB@1, IC4.VSSA, IC4.VSS_1, IC4.VSS_2, IC4.VSS_3, PAD2.P, R10.P$2, R15.P$2, R8.P$2; no longer C10.P$1, C11.P$2, C12.P$2, C16.P$1, C17.P$1, C20.P$1, C7.P$2, IC1.VSSA, IC1.VSS_1, IC1.VSS_2, IC1.VSS_3, IC2.CLKIN, IC2.FSYNC, IC3.CSB@1, IC4.GND, IC6.BOOT0, PAD15.P, R11.P$2, R12.P$2
- net M1+: now also PAD11.P; no longer PAD1.P
- net M2+: now also PAD15.P, Q3.D; no longer PAD2.P, Q2.D
- net M3+: now also PAD13.P, Q2.D; no longer PAD5.P, Q3.D
- net M4+: now also PAD17.P; no longer PAD6.P
- net MAIN_RX: now also IC4.PA10; no longer IC1.PA10
- net MAIN_TX: now also IC4.PA9, R12.P$2; no longer IC1.PA9, R14.P$2
- net N$1: now also IC1.INT, IC4.PA3, R9.P$1; no longer IC1.PA3, IC2.INT, R16.P$1
- net N$10: now also IC4.PB13, IC5.SCK; no longer IC1.PB13, IC4.SCK
- net N$11: now also IC4.PB14, IC5.MISO; no longer IC1.PB14, IC4.MISO
- net N$12: now also IC4.PB15, IC5.MOSI; no longer IC1.PB15, IC4.MOSI
- net N$13: now also IC4.PD1/OSC_OUT; no longer IC1.PD1/OSC_OUT
- net N$15: now also IC4.PB3, R16.P$1; no longer IC1.PB3, R6.P$1
- net N$16: now also R16.P$2; no longer R6.P$2
- net N$17: now also IC4.PC14/OSC32_IN, R7.P$2, R8.P$1; no longer IC1.PC14/OSC32_IN, R10.P$2, R11.P$1
- net N$18: now also R2.P$2; no longer R8.P$2
- net N$19: now also IC4.BOOT0, R15.P$1; no longer IC1.BOOT0, R12.P$1
- net N$2: now also IC1.CS, IC4.PA4, R5.P$1; no longer IC1.PA4, IC2.CS, R2.P$1
- net N$20: now also R1.P$2; no longer R7.P$2
- net N$24: now also R11.P$2; no longer R15.P$2
- net N$25: now also IC6.PA6
- net N$27: now also R12.P$1; no longer R14.P$1
- net N$3: now also IC1.SCL/SCLK, IC4.PA5; no longer IC1.PA5, IC2.SCL/SCLK
- net N$30: now also PAD8.P; no longer PAD10.P
- net N$31: now also R11.P$1; no longer R15.P$1
- net N$32: now also C4.P$2, IC1.REGOUT; no longer C15.P$2, IC2.REGOUT
- net N$33: now also IC4.PD0/OSC_IN; no longer IC1.PD0/OSC_IN
- net N$34: now also C5.P$2, IC1.CPOUT; no longer C17.P$2, IC2.CPOUT
- net N$35: now also IC4.PA1, PAD7.P; no longer IC1.PA1, PAD11.P
- net N$36: now also IC3.VI; no longer IC5.VI
- net N$37: now also C8.P$2, IC4.NRST; no longer C20.P$2, IC1.NRST
- net N$38: now also C11.P$2; no longer C8.P$2
- net N$4: now also IC1.AD0/SDO, IC4.PA6; no longer IC1.PA6, IC2.AD0/SDO
- net N$5: now also IC1.SDA/SDI, IC4.PA7; no longer IC1.PA7, IC2.SDA/SDI
- net N$6: now also IC4.PA0-WKUP; no longer IC1.PA0-WKUP
- net N$9: now also IC4.PB12, IC5.CS, R14.P$1; no longer IC1.PB12, IC4.CS, R3.P$1
- net PWM1: now also IC4.PB9; no longer IC1.PB9
- net PWM2: now also IC4.PB8, Q3.G, R19.P$2; no longer IC1.PB8, Q2.G, R18.P$2
- net PWM3: now also IC4.PB7, Q2.G, R18.P$2; no longer IC1.PB7, Q3.G, R19.P$2
- net PWM4: now also IC4.PA8; no longer IC1.PA8
- net SWCLK: now also IC4.PA14, PAD5.P; no longer IC1.PA14, PAD16.P
- net SWDIO: now also IC4.PA13, PAD6.P; no longer IC1.PA13, PAD17.P
- net USB_DM: now also IC4.PA11, R2.P$1; no longer IC1.PA11, R8.P$1
- net USB_DP: now also IC4.PA12, R1.P$1, R3.P$2; no longer IC1.PA12, R7.P$1, R9.P$2
- net VBUS: now also R7.P$1; no longer R10.P$1
- net VCC: now also C10.P$1, C12.P$2, C13.P$2, C14.P$2, C15.P$2, C16.P$1, C17.P$1, C7.P$2, C9.P$2, IC3.VO, IC4.VBAT, IC4.VDDA, IC4.VDD_1, IC4.VDD_2, IC4.VDD_3, IC5.HOLD, IC5.VCC, IC5.WP, PAD1.P, R14.P$2, R3.P$1, R6.P$2, R9.P$2; no longer C11.P$1, C12.P$1, C19.P$2, C2.P$2, C3.P$2, C4.P$2, C5.P$2, C6.P$2, C7.P$1, IC1.VBAT, IC1.VDDA, IC1.VDD_1, IC1.VDD_2, IC1.VDD_3, IC4.HOLD, IC4.VCC, IC4.WP, IC5.VO, PAD14.P, R16.P$2, R2.P$2, R3.P$2, R9.P$1
- net V_BARO: now also C1.P$2, C6.P$2, IC2.PS, IC2.VDD; no longer C10.P$2, C9.P$2, IC3.PS, IC3.VDD
- net V_GYRO: now also C2.P$2, C3.P$2, IC1.VDD; no longer C16.P$2, C18.P$2, IC2.VDD
Other:
- moved on the sheet: C10, C11, C12, C13, C14, C15, C16, C17, C18, C19, C2, C3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

Commit message: add BOM
Parts:
- 3V3: value VCC -> (none)
- D1: value (none) -> BAT54
- GND: value GND -> (none)
- IC1: value MPU-6050 -> MPU-6000
- IC3: value MCP1703CB -> XC6206P332
- IC5: value SPI_FLASH-X25XXSMD -> M25P16
- JP1: value M021X02_NO_SILK -> BAT
- PPM: value PPM -> (none)
- Q1, Q2, Q3, Q4: value (none) -> Si2312
- Q5: value (none) -> AO3401
- RX/SDA: value RX/SDA -> (none)
- SJ1: value JUMPER-PAD-2-NC_BY_PASTE -> BOOT
- SWCLK, SWCLK_: value SWCLK -> (none)
- SWDIO, SWDIO_: value SWDIO -> (none)
- TX/SCL: value TX/SCL -> (none)
- U$1: value UNTITLED_USB_AB -> microUSB
- renumbered PAD1 to 3V3, PAD10 to M1+, PAD11 to M1-, PAD12 to M3+, PAD13 to M3-, PAD14 to M2+, PAD15 to M2-, PAD16 to M4+, PAD17 to M4-, PAD2 to GND, PAD3 to RX/SDA, PAD4 to TX/SCL, PAD5 to SWCLK_, PAD6 to SWDIO_, PAD7 to PPM, PAD8 to SWCLK, PAD9 to SWDIO, T1 to Q5
